File: ergogen/output/pcbs/regret.kicad_pcb (KiCad board)
At the start: 2 copper layers, 227.4 x 104.4 mm, 93 parts

Commit message: Embrace `mirror` for LED layout
Parts:
- moved LED4 157.1 mm to (256.3, 100.1), turned to 9 degrees
- moved LED2 141.1 mm to (208.8, 100.0), turned to 20 degrees
- moved LED9 130.6 mm to (132.2, 152.7), turned to -20 degrees
- moved LED6 109.6 mm to (259.6, 117.3), turned to 9 degrees
- moved LED7 89.3 mm to (102.9, 133.8)
- moved LED10 82.0 mm to (191.8, 152.7), turned to 20 degrees
- moved LED11 79.8 mm to (162.0, 165.8), turned to 0 degrees
- moved LED5 76.4 mm to (64.5, 117.3), turned to -9 degrees
- moved LED3 17.5 mm to (67.8, 100.1)
- moved D16 1.59 mm to (265.1, 132.8)
- moved D17 1.59 mm to (262.4, 116.0)
- moved D18 1.59 mm to (259.7, 99.2)
- moved D19 1.59 mm to (245.8, 128.9)
- moved D20 1.59 mm to (241.1, 112.6)
- moved D21 1.59 mm to (236.4, 96.2)
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Connections:
- LED10 pad 2: L11 -> L8
- LED10 pad 4: L10 -> L7
- LED11 pad 2: (no net) -> L7
- LED11 pad 4: L11 -> L6
- LED2 pad 2: L3 -> (no net)
- LED2 pad 4: L2 -> L11
- LED3 pad 2: L4 -> L3
- LED3 pad 4: L3 -> L2
- LED4 pad 2: L5 -> L11
- LED4 pad 4: L4 -> L10
- LED5 pad 2: L6 -> L4
- LED5 pad 4: L5 -> L3
- LED6 pad 2: L7 -> L10
- LED6 pad 4: L6 -> L9
- LED7 pad 2: L8 -> L5
- LED7 pad 4: L7 -> L4
- LED9 pad 2: L10 -> L6
- LED9 pad 4: L9 -> L5
Other:
- board size 227.4 x 104.4 mm -> 229 x 104.4 mm

Commit message: Add sacrificial diode to LED1
Parts:
- added D35: , ComboDiode, F.Cu at (116.3, 97.2)
- LED1, LED10, LED11, LED2, LED3, LED4, LED5, LED6, LED7, LED8, LED9: value VAL** -> SK6812-MINI-E; footprint WS2812B -> SK6812-MINI-E
Connections:
- LED1 pad 1: VUSB -> led_1_v

Commit message: v1.0.0
Parts:
- added B1: , Panasonic_EVQPUL_EVQPUC, B.Cu at (171.6, 107.7)
- added JST1: , JST_PH_S2B-PH-K_02x2.00mm_Angled, F.Cu at (152.8, 148.0)
- added SB1: , ChocBonusGoodies, F.Cu at (59.8, 128.2)
- added SB10: , ChocBonusGoodies, F.Cu at (114.5, 134.2)
- added SB11: , ChocBonusGoodies, F.Cu at (120.3, 118.2)
- added SB12: , ChocBonusGoodies, F.Cu at (126.2, 102.2)
- added SB13: , ChocBonusGoodies, F.Cu at (130.6, 142.6)
- added SB14: , ChocBonusGoodies, F.Cu at (136.4, 126.6)
- added SB15: , ChocBonusGoodies, F.Cu at (142.3, 110.6)
- added SB16: , ChocBonusGoodies, F.Cu at (264.3, 128.2)
- added SB17: , ChocBonusGoodies, F.Cu at (261.7, 111.4)
- added SB18: , ChocBonusGoodies, F.Cu at (259.0, 94.6)
- added SB19: , ChocBonusGoodies, F.Cu at (244.5, 124.4)
- added SB2: , ChocBonusGoodies, F.Cu at (62.4, 111.4)
- added SB20: , ChocBonusGoodies, F.Cu at (239.8, 108.0)
- added SB21: , ChocBonusGoodies, F.Cu at (235.1, 91.7)
- added SB22: , ChocBonusGoodies, F.Cu at (225.3, 124.8)
- added SB23: , ChocBonusGoodies, F.Cu at (219.5, 108.9)
- added SB24: , ChocBonusGoodies, F.Cu at (213.7, 92.9)
- added SB25: , ChocBonusGoodies, F.Cu at (209.6, 134.2)
- added SB26: , ChocBonusGoodies, F.Cu at (203.8, 118.2)
- added SB27: , ChocBonusGoodies, F.Cu at (197.9, 102.2)
- added SB28: , ChocBonusGoodies, F.Cu at (193.5, 142.6)
- added SB29: , ChocBonusGoodies, F.Cu at (187.7, 126.6)
- added SB3: , ChocBonusGoodies, F.Cu at (65.1, 94.6)
- added SB30: , ChocBonusGoodies, F.Cu at (181.8, 110.6)
- added SB31: , ChocBonusGoodies, F.Cu at (123.4, 159.1)
- added SB32: , ChocBonusGoodies, F.Cu at (139.8, 168.8)
- added SB33: , ChocBonusGoodies, F.Cu at (200.7, 159.1)
- added SB34: , ChocBonusGoodies, F.Cu at (184.3, 168.8)
- added SB4: , ChocBonusGoodies, F.Cu at (79.6, 124.4)
- added SB5: , ChocBonusGoodies, F.Cu at (84.3, 108.0)
- added SB6: , ChocBonusGoodies, F.Cu at (88.9, 91.7)
- added SB7: , ChocBonusGoodies, F.Cu at (98.8, 124.8)
- added SB8: , ChocBonusGoodies, F.Cu at (104.6, 108.9)
- added SB9: , ChocBonusGoodies, F.Cu at (110.4, 92.9)
- added T1: , E73:SPDT_C128955, F.Cu at (161.5, 123.6)
- LED1, LED10, LED11, LED2, LED3, LED4, LED5, LED6, LED7, LED8, LED9: value SK6812-MINI-E -> VAL**; footprint SK6812-MINI-E -> WS2812B
- moved D35 3.61 mm to (119.8, 96.3)
- moved LED10 2.00 mm to (191.2, 150.8)
- moved LED9 2.00 mm to (132.9, 150.8)
- moved MCU1 1.00 mm to (162.0, 134.1)
Other:
- board size 229 x 104.4 mm -> 229 x 107.1 mm
